File: PCB/_autosave-PCB.kicad_sch (KiCad schematic)
At the start: 10 parts, among them SW1 Bourns PEC11R, SW2 Bourns PEC11R, SW3 SW_DPST, SW4 SW_DPST, SW5 SW_DPST, U1 RPi_Pico_TH, U2 RDA5807M_Module, U3 LM386

Commit message: kicad lab experiment and initial draft of schematic
Other:
- note added: "0"
- note added: "Watering hole clock radio"
Changed lines of the file:
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@@
 	(generator_version "9.0")
 	(paper "A4")
+	(text "0"
+		(exclude_from_sim no)
+		(at 268.732 193.548 0)
+		(effects
+			(font
+				(size 1.27 1.27)
+			)
+		)
+	)
+	(text "Watering hole clock radio"
+		(exclude_from_sim no)
+		(at 198.882 189.992 0)
+		(effects
+			(font
+				(size 1.27 1.27)
+			)
+		)
+	)
 	(junction
 		(at 50.8 85.09)
