File: PCB/PCB.kicad_sch (KiCad schematic)
At the start: 38 parts, among them SW1 Bourns PEC11R, SW2 Bourns PEC11R, SW3 SW_DPST, SW4 SW_DPST, SW5 SW_DPST, U1 RPi_Pico_TH, U2 RDA5807M_Module, U3 LM386, U4 AP63205WU-7

Commit message: changed sw5 footprint to button footprint
Parts:
- SW5: footprint 2pin_ScrewTerminal:691137710002 -> Button_Switch_THT:SW_PUSH_6mm_H7.3mm
Changed lines of the file:
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@@
 			)
 		)
-		(property "Footprint" "2pin_ScrewTerminal:691137710002"
+		(property "Footprint" "Button_Switch_THT:SW_PUSH_6mm_H7.3mm"
 			(at 148.59 130.81 0)
 			(effects

Commit message: code and some stl
Connections:
- net GND: now also C3.1, U3.2 (-)
- net Radio sclk: now also U1.27 (GP21); no longer U1.26 (GP20)
- net Radio sdio: now also U1.26 (GP20); no longer U1.27 (GP21)
Changed lines of the file:
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@@
+	)
+	(junction
+		(at 160.02 54.61)
+		(diameter 0)
+		(color 0 0 0 0)
 	)
 	(junction
@@
 	)
 	(junction
+		(at 170.18 62.23)
+		(diameter 0)
+		(color 0 0 0 0)
+	)
+	(junction
 		(at 114.3 186.69)
 		(diameter 0)
@@
 	(wire
 		(pts
+			(xy 160.02 54.61) (xy 160.02 62.23)
+		)
+		(stroke
+			(width 0)
+			(type default)
+		)
+	)
+	(wire
+		(pts
 			(xy 52.07 44.45) (xy 52.07 39.37)
 		)
@@
 	(wire
 		(pts
-			(xy 170.18 59.69) (xy 170.18 64.77)
+			(xy 170.18 59.69) (xy 170.18 62.23)
 		)
 		(stroke
@@
 	(wire
 		(pts
+			(xy 170.18 62.23) (xy 170.18 64.77)
+		)
+		(stroke
+			(width 0)
+			(type default)
+		)
+	)
+	(wire
+		(pts
 			(xy 100.33 167.64) (xy 111.76 167.64)
 		)
@@
 		(pts
 			(xy 15.24 29.21) (xy 15.24 30.48)
+		)
+		(stroke
+			(width 0)
+			(type default)
+		)
+	)
+	(wire
+		(pts
+			(xy 160.02 62.23) (xy 170.18 62.23)
 		)
 		(stroke
@@
 	)
 	(label "Radio sclk"
-		(at 64.77 80.01 0)
+		(at 64.77 77.47 0)
 		(effects
 			(font
@@
 	)
 	(label "Radio sdio"
-		(at 64.77 77.47 0)
-		(effects
-			(font
+		(at 64.77 80.01 0)
+		(effects
+			(font
